File: ESP32_BUCK_WLED_NO_BOARD.kicad_pcb (KiCad board)
At the start: 2 copper layers, 55.9 x 77.5 mm, 37 parts, among them J2 LEDSTRIPS_DATA_ALIMENTATIION, J3 BOARD_ALIMENTATION, J5 ESP_FLASH_PIN, J6 Conn_01x02, Q1 SS8050, Q2 SS8050, SW2 SW_Push, SW3 SW_Push, U1 LM2596T-ADJ, U2 AMS1117-3.3, U3 ESP32-WROOM-32E, U5 74AHCT125

Commit message: final version with gerber files
Parts:
- moved J6 2.54 mm to (142.2, 71.1)
- renumbered C2 to C1, C6 to C10, C7 to C5, C16 to C6, C5 to C7, R6 to R11, R7 to R12, R8 to R13, R9 to R14, R2 to R4, R3 to R5, R4 to R6, R5 to R7, R15 to R9
Routing:
- net /EN: track 0.00 -> 80.4 mm, vias 0 -> 5
- net /IO16: track 0.00 -> 56.1 mm, vias 0 -> 2
- net /IO17: track 0.00 -> 54.2 mm, vias 0 -> 2
- net /IO19: track 0.00 -> 53.6 mm, vias 0 -> 2
- net /IO18: track 0.00 -> 50.7 mm, vias 0 -> 2
- net /RTS: track 2.81 -> 45.2 mm, vias 0 -> 1
- net /DTR: track 3.35 -> 42.3 mm, vias 0 -> 1
- net /IO0: track 0.00 -> 37.5 mm, vias 0 -> 2
- net /RXD0: track 0.00 -> 37.3 mm, vias 0 -> 1
- net /RXD: track 0.00 -> 36.7 mm, vias 0 -> 1
- net Net-(R4-Pad2): track 0.00 -> 18.8 mm, vias 0 -> 1
- net Net-(U1-FB): track 0.00 -> 15.4 mm, vias 0 -> 2
- net /LED1: track 0.00 -> 15.2 mm, vias 0 -> 2
- net Net-(D1-K): track 0.00 -> 14.8 mm, vias 0 -> 2
- net /VDD33: track 0.00 -> 14.6 mm, vias 0 -> 5
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- added copper zone on B.Cu, net /5V_BUCK
- added copper zone on B.Cu, net /5V_ESP
- added copper zone on B.Cu, net /VDD33
- added copper zone on B.Cu, net /V_ALIM
- added copper zone on F.Cu, net GND
Other:
- board size 55.9 x 77.5 mm -> 55.9 x 78.7 mm
- copper layers 2 -> 4
- board text added: "github.com/ lepetidozo/ wledController_V1"

Commit message: Add files via upload
added test points
Parts:
- added TP1: TestPoint, TestPoint:TestPoint_Pad_D1.5mm, F.Cu at (134.6, 99.1)
- added TP2: TestPoint, TestPoint:TestPoint_Pad_D1.5mm, F.Cu at (137.2, 99.1)
- added TP3: TestPoint, TestPoint:TestPoint_Pad_D1.5mm, F.Cu at (132.1, 76.2)
- added TP4: TestPoint, TestPoint:TestPoint_Pad_D1.5mm, F.Cu at (137.2, 76.2)
- added TP5: TestPoint, TestPoint:TestPoint_Pad_D1.5mm, F.Cu at (137.2, 68.6)
- added TP6: TestPoint, TestPoint:TestPoint_Pad_D1.5mm, F.Cu at (147.3, 68.6)
Routing:
- net /VDD33: track 14.6 -> 8.28 mm
Other:
- board text added: "BOOT"
- board text added: "EN"
- board text added: "GND"
- board text added: "VIN"
