File: ESP32_BUCK_WLED_NO_BOARD.kicad_sch (KiCad schematic)
At the start: 50 parts, among them J1 USB_C_Receptacle_USB2.0_16P, J2 LEDSTRIPS_DATA_ALIMENTATIION, J3 BOARD_ALIMENTATION, J4 Conn_01x03, J5 ESP_FLASH_PIN, J6 Conn_01x02, Q1 SS8050, Q2 SS8050, SW2 SW_Push, SW3 SW_Push, U1 LM2596T-ADJ, U2 AMS1117-3.3, U3 ESP32-WROOM-32E, U4 CP2102N-A02-GQFN28, U5 74AHCT125

Commit message: final version with gerber files
Parts:
- renumbered C2 to C1, C6 to C10, C10 to C2, C7 to C5, C16 to C6, C5 to C7, R17 to R10, R6 to R11, R7 to R12, R8 to R13, R9 to R14, R10 to R15, R14 to R16, R12 to R2, R13 to R3, R2 to R4, R3 to R5, R4 to R6, R5 to R7, R11 to R8, R15 to R9
Changed lines of the file:
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@@
 		(in_pos_files yes)
 		(dnp no)
-		(property "Reference" "C7"
+		(property "Reference" "C5"
 			(at 18.034 86.36 0)
 			(show_name no)
@@
 			(project "ESP32_BUCK_WLED_NO_BOARD"
 				(path "/825652b8-9479-497b-b5c8-f7254daf27f6"
-					(reference "C7")
+					(reference "C5")
 					(unit 1)
 				)
@@
 		(in_pos_files yes)
 		(dnp no)
-		(property "Reference" "R8"
+		(property "Reference" "R13"
 			(at 219.456 139.7 90)
 			(show_name no)
@@
 			(project "ESP32_BUCK_WLED_NO_BOARD"
 				(path "/825652b8-9479-497b-b5c8-f7254daf27f6"
-					(reference "R8")
+					(reference "R13")
 					(unit 1)
 				)
@@
 		(in_pos_files yes)
 		(dnp no)
-		(property "Reference" "R9"
+		(property "Reference" "R14"
 			(at 219.456 137.16 90)
 			(show_name no)
@@
 			(project "ESP32_BUCK_WLED_NO_BOARD"
 				(path "/825652b8-9479-497b-b5c8-f7254daf27f6"
-					(reference "R9")
+					(reference "R14")
 					(unit 1)
 				)
@@
 		(in_pos_files yes)
 		(dnp no)
-		(property "Reference" "R15"
+		(property "Reference" "R9"
 			(at 19.05 111.76 0)
 			(show_name no)
@@
 			(project "ESP32_BUCK_WLED_NO_BOARD"
 				(path "/825652b8-9479-497b-b5c8-f7254daf27f6"
-					(reference "R15")
+					(reference "R9")
 					(unit 1)
 				)
@@
 		(in_pos_files yes)
 		(dnp yes)
-		(property "Reference" "R10"
+		(property "Reference" "R15"
 			(at 88.646 120.396 90)
 			(show_name no)
@@
 			(project "ESP32_BUCK_WLED_NO_BOARD"
 				(path "/825652b8-9479-497b-b5c8-f7254daf27f6"
-					(reference "R10")
+					(reference "R15")
 					(unit 1)
 				)
@@
 		(in_pos_files yes)
 		(dnp no)
-		(property "Reference" "C5"
+		(property "Reference" "C7"
 			(at 196.342 31.242 90)
 			(show_name no)
@@
 			(project "ESP32_BUCK_WLED_NO_BOARD"
 				(path "/825652b8-9479-497b-b5c8-f7254daf27f6"
-					(reference "C5")
+					(reference "C7")
 					(unit 1)
 				)
@@
 		(in_pos_files yes)
 		(dnp no)
-		(property "Reference" "R6"
+		(property "Reference" "R11"
 			(at 219.456 144.78 90)
 			(show_name no)
@@
 			(project "ESP32_BUCK_WLED_NO_BOARD"
 				(path "/825652b8-9479-497b-b5c8-f7254daf27f6"
-					(reference "R6")
+					(reference "R11")
 					(unit 1)
 				)
@@
 		(in_pos_files yes)
 		(dnp no)
-		(property "Reference" "R4"
+		(property "Reference" "R6"
 			(at 222.758 24.13 90)
 			(show_name no)
@@
 			(project "ESP32_BUCK_WLED_NO_BOARD"
 				(path "/825652b8-9479-497b-b5c8-f7254daf27f6"
-					(reference "R4")
+					(reference "R6")
 					(unit 1)
 				)
@@
 		(in_pos_files yes)
 		(dnp yes)
-		(property "Reference" "R12"
+		(property "Reference" "R2"
 			(at 182.118 92.456 90)
 			(show_name no)
@@
 			(project "ESP32_BUCK_WLED_NO_BOARD"
 				(path "/825652b8-9479-497b-b5c8-f7254daf27f6"
-					(reference "R12")
+					(reference "R2")
 					(unit 1)
 				)
@@
 		(in_pos_files yes)
 		(dnp no)
-		(property "Reference" "C6"
+		(property "Reference" "C10"
 			(at 196.088 56.388 90)
 			(show_name no)
@@
 			(project "ESP32_BUCK_WLED_NO_BOARD"
 				(path "/825652b8-9479-497b-b5c8-f7254daf27f6"
-					(reference "C6")
+					(reference "C10")
 					(unit 1)
 				)
@@
 		(in_pos_files yes)
 		(dnp yes)
-		(property "Reference" "R17"
+		(property "Reference" "R10"
 			(at 112.522 100.838 0)
 			(show_name no)
@@
 			(project "ESP32_BUCK_WLED_NO_BOARD"
 				(path "/825652b8-9479-497b-b5c8-f7254daf27f6"
-					(reference "R17")
+					(reference "R10")
 					(unit 1)
 				)
@@
 		(in_pos_files yes)
 		(dnp no)
-		(property "Reference" "R2"
+		(property "Reference" "R4"
 			(at 104.648 47.498 0)
 			(show_name no)
@@
 			(project "ESP32_BUCK_WLED_NO_BOARD"
 				(path "/825652b8-9479-497b-b5c8-f7254daf27f6"
-					(reference "R2")
+					(reference "R4")
 					(unit 1)
 				)
@@
 		(in_pos_files yes)
 		(dnp no)
-		(property "Reference" "R7"
+		(property "Reference" "R12"
 			(at 219.456 142.24 90)
 			(show_name no)
@@
 			(project "ESP32_BUCK_WLED_NO_BOARD"
 				(path "/825652b8-9479-497b-b5c8-f7254daf27f6"
-					(reference "R7")
+					(reference "R12")
 					(unit 1)
 				)
@@
 		(in_pos_files yes)
 		(dnp no)
-		(property "Reference" "R5"
+		(property "Reference" "R7"
 			(at 222.758 38.1 90)
 			(show_name no)
@@
 			(project "ESP32_BUCK_WLED_NO_BOARD"
 				(path "/825652b8-9479-497b-b5c8-f7254daf27f6"
-					(reference "R5")
+					(reference "R7")
 					(unit 1)
 				)
@@
 		(in_pos_files yes)
 		(dnp yes)
-		(property "Reference" "R13"
+		(property "Reference" "R3"
 			(at 182.372 98.044 90)
 			(show_name no)
@@
 			(project "ESP32_BUCK_WLED_NO_BOARD"
 				(path "/825652b8-9479-497b-b5c8-f7254daf27f6"
-					(reference "R13")
+					(reference "R3")
 					(unit 1)
 				)
@@
 		(in_pos_files yes)
 		(dnp yes)
-		(property "Reference" "R14"
+		(property "Reference" "R16"
 			(at 99.568 123.444 0)
 			(show_name no)
@@
 			(project "ESP32_BUCK_WLED_NO_BOARD"
 				(path "/825652b8-9479-497b-b5c8-f7254daf27f6"
-					(reference "R14")
+					(reference "R16")
 					(unit 1)
 				)
@@
 		(in_pos_files yes)
 		(dnp yes)
-		(property "Reference" "C10"
+		(property "Reference" "C2"
 			(at 94.234 87.63 0)
 			(show_name no)
@@
 			(project "ESP32_BUCK_WLED_NO_BOARD"
 				(path "/825652b8-9479-497b-b5c8-f7254daf27f6"
-					(reference "C10")
+					(reference "C2")
 					(unit 1)
 				)
@@
 		(in_pos_files yes)
 		(dnp no)
-		(property "Reference" "R3"
+		(property "Reference" "R5"
 			(at 154.178 53.848 0)
 			(show_name no)
@@
 			(project "ESP32_BUCK_WLED_NO_BOARD"
 				(path "/825652b8-9479-497b-b5c8-f7254daf27f6"
-					(reference "R3")
+					(reference "R5")
 					(unit 1)
 				)
@@
 		(in_pos_files yes)
 		(dnp no)
-		(property "Reference" "C16"
+		(property "Reference" "C6"
 			(at 258.318 148.59 90)
 			(show_name no)
@@
 			(project "ESP32_BUCK_WLED_NO_BOARD"
 				(path "/825652b8-9479-497b-b5c8-f7254daf27f6"
-					(reference "C16")
+					(reference "C6")
 					(unit 1)
 				)
@@
 		(in_pos_files yes)
 		(dnp yes)
-		(property "Reference" "R11"
+		(property "Reference" "R8"
 			(at 144.018 125.476 0)
 			(show_name no)
@@
 			(project "ESP32_BUCK_WLED_NO_BOARD"
 				(path "/825652b8-9479-497b-b5c8-f7254daf27f6"
-					(reference "R11")
+					(reference "R8")
 					(unit 1)
 				)
@@
 		(in_pos_files yes)
 		(dnp no)
-		(property "Reference" "C2"
+		(property "Reference" "C1"
 			(at 88.138 44.196 0)
 			(show_name no)
@@
 			(project "ESP32_BUCK_WLED_NO_BOARD"
 				(path "/825652b8-9479-497b-b5c8-f7254daf27f6"
-					(reference "C2")
+					(reference "C1")
 					(unit 1)
 				)

Commit message: Add files via upload
added test points
Parts:
- added TP1, TP2, TP3, TP4, TP5, TP6: TestPoint, TestPoint:TestPoint_Pad_D1.5mm, symbol Connector:TestPoint
Connections:
- net 5V_BUCK: now also TP3.1
- net GND: now also TP2.1, TP4.1, TP6.1
- net VDD33: now also TP5.1
- net V_ALIM: now also TP1.1
Other:
- moved on the sheet: C14, C15, J3
